File: NukeNanny.sch (EAGLE design)
At the start: 46 parts, among them IC1 25AA080SN, Q1 MMBT4403, U1 CR2032, U2 SHT1XSMD, U3 HX711

Commit message: Changed sensor to HTU21D
Parts:
- removed U2: SHT1XSMD, SparkFun-Sensors:SHT1XSMD
- added R13, R16: 1k, rcl:R-US_R0805
- added U4: HTU21D, SparkFun-Sensors:HTU21DSMD
- C11: value 6.8p -> 0.1u
- C9: value 3.3 -> 3.3p
- R1, R2: value (none) -> 200
Connections:
- net GND: now also U4.GND@2, U4.GND@7; no longer U2.GND
- net SHDAT: now also R13.2, U4.DATA; no longer U2.DATA
- net SHSCK: now also R16.2, U4.SCK; no longer U2.SCK
- net VCC: now also R13.1, R16.1, U4.VDD; no longer U2.VDD
